File: PCBS/Boards/Tenn/Tenn.kicad_sch (KiCad schematic)
At the start: 29 parts, among them J1 Conn_01x02_Socket, J12 Conn_01x04_Female, J13 Conn_01x03_Male, J14 Conn_01x03_Male, J15 Conn_01x03_Male, J16 Conn_01x02_Male, J17 Conn_01x02_Male, J18 Conn_01x30_Pin, SW2 SW_Push, SW3 SW_Push, SW4 SW_SPDT, U1 L7805, U2 DRV8871DDA, U3 DRV8871DDA

Commit message: updates files of tenn pcb, changes foot print of 47uf capacitor, fixes unconnected vias and traces, adds Arduino GPIO references in the backside for easier understanding of the board
Parts:
- C5, C6: footprint Capacitor_SMD:C_0805_2012Metric_Pad1.18x1.45mm_HandSolder -> Capacitor_SMD:C_1206_3216Metric_Pad1.33x1.80mm_HandSolder
Changed lines of the file:
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@@
 			)
 		)
-		(property "Footprint" "Capacitor_SMD:C_0805_2012Metric_Pad1.18x1.45mm_HandSolder"
+		(property "Footprint" "Capacitor_SMD:C_1206_3216Metric_Pad1.33x1.80mm_HandSolder"
 			(at 244.8052 109.22 0)
 			(effects
@@
 			)
 		)
-		(property "Footprint" "Capacitor_SMD:C_0805_2012Metric_Pad1.18x1.45mm_HandSolder"
+		(property "Footprint" "Capacitor_SMD:C_1206_3216Metric_Pad1.33x1.80mm_HandSolder"
 			(at 244.8052 146.05 0)
 			(effects
