File: PCBS/Boards/Tenn/Tenn.kicad_sch (KiCad schematic)
At the start: 29 parts, among them J1 Conn_01x02_Socket, J12 Conn_01x04_Female, J13 Conn_01x03_Male, J14 Conn_01x03_Male, J15 Conn_01x03_Male, J16 Conn_01x02_Male, J17 Conn_01x02_Male, J18 Conn_01x30_Pin, SW2 SW_Push, SW3 SW_Push, SW4 SW_SPDT, U1 L7805, U2 DRV8871DDA, U3 DRV8871DDA

Commit message: created SHU BEC, added KiCad project files and production files
Parts:
- removed J1: Conn_01x02_Socket, Connector_AMASS:AMASS_XT30U-M_1x02_P5.0mm_Vertical, symbol Connector:Conn_01x02_Socket
- removed J12: Conn_01x04_Female, Connector_PinSocket_2.54mm:PinSocket_1x04_P2.54mm_Vertical, symbol Connector:Conn_01x04_Female
- removed J13, J14: Conn_01x03_Male, Connector_PinSocket_2.54mm:PinSocket_1x03_P2.54mm_Vertical, symbol Connector:Conn_01x03_Male
- removed J15: Conn_01x03_Male, Connector_PinHeader_2.54mm:PinHeader_1x03_P2.54mm_Vertical, symbol Connector:Conn_01x03_Male
- removed J16, J17: Conn_01x02_Male, Connector_JST:JST_XH_B2B-XH-A_1x02_P2.50mm_Vertical, symbol Connector:Conn_01x02_Male
- added J1: XT30 Male, Connector_AMASS:AMASS_XT30U-M_1x02_P5.0mm_Vertical, symbol Connector_Generic:Conn_01x02
- added J3, J6: Conn_01x04, Connector_PinSocket_2.54mm:PinSocket_1x04_P2.54mm_Vertical, symbol Connector_Generic:Conn_01x04
- added J4: Conn_01x03, Connector_PinSocket_2.54mm:PinSocket_1x03_P2.54mm_Vertical, symbol Connector_Generic:Conn_01x03
- added J5: Conn_01x03, Connector_PinHeader_2.54mm:PinHeader_1x03_P2.54mm_Vertical, symbol Connector_Generic:Conn_01x03
- added J8, J9: Conn_01x02, Connector_JST:JST_XH_B2B-XH-A_1x02_P2.50mm_Vertical, symbol Connector_Generic:Conn_01x02
- added SW4: SW_Push, Button_Switch_SMD:SW_SPST_B3U-1000P, symbol Switch:SW_Push
- added TP1, TP2, TP3: TestPoint, PCM_SparkFun-Connector:TestPoint-0.75mm, symbol Connector:TestPoint
- added U4: MATEKSYS_MICRO_BEC, Custom Development Boards:MATEKSYS MICRO BEC, symbol DIY modules:MATEKSYS_MICRO_BEC
- C1, C2: symbol Device:C -> Device:C_Small
- C3: renamed from C6; symbol Device:C -> Device:C_Small
- C4: renamed from C5; symbol Device:C -> Device:C_Small
- C5: renamed from C4; symbol Device:C -> Device:C_Small
- C6: renamed from C3; symbol Device:C -> Device:C_Small
- R1: renamed from R2; symbol Device:R -> Device:R_Small
- R2: renamed from R1; symbol Device:R -> Device:R_Small
- R3: renamed from R4; symbol Device:R -> Device:R_Small
- R4: renamed from R3; symbol Device:R -> Device:R_Small
- renumbered J18 to J2, SW4 to SW1, SW3 to SW2, SW2 to SW3, U3 to U2, U2 to U3
Connections:
- net VCC is gone; now on net +5V: A1.30 (VIN), C2.1, U1.3 (OUT)
- net +3.3V: now also TP1.1
- net +5V: now also J3.3 (Pin_3), J4.1 (Pin_1), J5.2 (Pin_2), J6.3 (Pin_3), TP2.1, U4.4 (VOUT); no longer A1.27 (+5V)
- net GND: now also C4.1, R3.2, R4.2, J1.1 (Pin_1), J3.4 (Pin_4), J4.2 (Pin_2), J5.3 (Pin_3), J6.4 (Pin_4), SW4.2, TP3.1, U4.2 (GNDIN), U4.3 (GND_OUT); no longer C4.2, R3.1, R4.1
- net MA1: now also U2.3 (IN1); no longer U2.2 (IN2)
- net MA2: now also U2.2 (IN2); no longer U2.3 (IN1)
- net MB1: now also U3.3 (IN1); no longer U3.2 (IN2)
- net MB2: now also U3.2 (IN2); no longer U3.3 (IN1)
- net SCL: now also J3.2 (Pin_2)
- net SDA: now also J3.1 (Pin_1)
- net Servo: now also J5.1 (Pin_1)
- net RX/D1: now reaches A1.1 (D1/TX)
- net RX/D1: now also J6.2 (Pin_2)
- net TX/D0: now reaches A1.2 (D0/RX)
- net TX/D0: now also J6.1 (Pin_1)
- net at A1.28 (~{RESET}): now also A1.3 (~{RESET}), SW4.1
- net at U2.4 (ILIM): now also R3.1; no longer R3.2
- net at U3.6 (OUT1): now also J9.1 (Pin_1)
- net at U3.8 (OUT2): now also J9.2 (Pin_2)
- net at SW1.1 (A): now also J1.2 (Pin_2)
- net at U3.4 (ILIM): now also R4.1; no longer R4.2
- net at U2.6 (OUT1): now also J8.1 (Pin_1)
- net at U2.8 (OUT2): now also J8.2 (Pin_2)
- net GO renamed Go
- net Go: now also J4.3 (Pin_3)
- net VM renamed +BATT
- net +BATT: now also C4.2, U4.1 (VIN); no longer C4.1
Other:
- note added: "Screen/I2C"
- note added: "TX/RX"
- note removed: "Screen"
- moved on the sheet: A1, C1, C2, C3, C4, C5, C6, H1, H2, H3, H4, J2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
