File: PCBS/Boards/Tenn/Tenn.kicad_pcb (KiCad board)
At the start: 2 copper layers, 85.5 x 24 mm, 66 parts, among them J1 Conn_01x02_Socket, J12 Conn_01x04_Female, J13 Conn_01x03_Male, J14 Conn_01x03_Male, J15 Conn_01x03_Male, J16 Conn_01x02_Male, J17 Conn_01x02_Male, J18 Conn_01x30_Pin, SW2 SW_Push, SW3 SW_Push, SW4 SW_SPDT, U1 L7805, U2 DRV8871DDA, U3 DRV8871DDA

Commit message: created SHU BEC, added KiCad project files and production files
Parts:
- removed 5V, G*** (x29), G1, G2, G3, G5, GND: LOGO, LOGO
- removed ANALOG IN: LOGO, LOGO
- removed DIGITAL IN: LOGO, LOGO
- removed J12: Conn_01x04_Female, Connector_PinSocket_2.54mm:PinSocket_1x04_P2.54mm_Vertical
- removed J13, J14: Conn_01x03_Male, Connector_PinSocket_2.54mm:PinSocket_1x03_P2.54mm_Vertical
- removed J15: Conn_01x03_Male, Connector_PinHeader_2.54mm:PinHeader_1x03_P2.54mm_Vertical
- removed J16, J17: Conn_01x02_Male, Connector_JST:JST_XH_B2B-XH-A_1x02_P2.50mm_Vertical
- removed J18: Conn_01x30_Pin, Connector_PinSocket_2.54mm:PinSocket_1x30_P2.54mm_Vertical
- added J2: Conn_01x30_Pin, Connector_PinSocket_2.54mm:PinSocket_1x30_P2.54mm_Vertical, F.Cu at (186.8, 89.2)
- added J3: Conn_01x04, Connector_PinSocket_2.54mm:PinSocket_1x04_P2.54mm_Vertical, F.Cu at (145.4, 96.2)
- added J4: Conn_01x03, Connector_PinSocket_2.54mm:PinSocket_1x03_P2.54mm_Vertical, F.Cu at (171.6, 110.8)
- added J5: Conn_01x03, Connector_PinHeader_2.54mm:PinHeader_1x03_P2.54mm_Vertical, F.Cu at (176.7, 110.8)
- added J6: Conn_01x04, Connector_PinSocket_2.54mm:PinSocket_1x04_P2.54mm_Vertical, F.Cu at (141.9, 96.2)
- added J8: Conn_01x02, Connector_JST:JST_XH_B2B-XH-A_1x02_P2.50mm_Vertical, F.Cu at (86.3, 115.3)
- added J9: Conn_01x02, Connector_JST:JST_XH_B2B-XH-A_1x02_P2.50mm_Vertical, F.Cu at (76.4, 115.3)
- added SW1: SW_SPDT, Button_Switch_THT:SW_Slide_SPDT_Straight_CK_OS102011MS2Q, F.Cu at (112.3, 100.5)
- added TP1: TestPoint, PCM_SparkFun-Connector:TestPoint-0.75mm, F.Cu at (113.2, 110.2)
- added TP2: TestPoint, PCM_SparkFun-Connector:TestPoint-0.75mm, F.Cu at (114.4, 110.2)
- added TP3: TestPoint, PCM_SparkFun-Connector:TestPoint-0.75mm, F.Cu at (115.7, 110.2)
- added U4: MATEKSYS_MICRO_BEC, Custom Development Boards:MATEKSYS MICRO BEC, B.Cu at (61.9, 102.4)
- C3, C4: value 0.1uF -> 47uF; footprint Capacitor_SMD:C_0805_2012Metric_Pad1.18x1.45mm_HandSolder -> Capacitor_SMD:C_1206_3216Metric_Pad1.33x1.80mm_HandSolder
- C5, C6: value 47uF -> 0.1uF; footprint Capacitor_SMD:C_1206_3216Metric_Pad1.33x1.80mm_HandSolder -> Capacitor_SMD:C_0805_2012Metric_Pad1.18x1.45mm_HandSolder
- J1: value Conn_01x02_Socket -> XT30 Male; moved to B.Cu
- SW4: value SW_SPDT -> SW_Push; footprint Button_Switch_THT:SW_Slide_SPDT_Straight_CK_OS102011MS2Q -> Button_Switch_SMD:SW_SPST_B3U-1000P
- moved SW4 94.9 mm to (205.4, 106.0), turned to 0 degrees
- moved U1 89.0 mm to (61.9, 102.4), turned to -90 degrees
- moved H3 87.3 mm to (191.0, 110.5)
- moved H4 76.3 mm to (109.0, 110.5)
- moved C2 59.9 mm to (66.4, 98.4), turned to -90 degrees
- moved C1 59.0 mm to (57.3, 98.4), turned to -90 degrees
- moved C3 51.8 mm to (74.9, 108.1), turned to 90 degrees
- moved C6 44.7 mm to (82.7, 108.1), turned to 90 degrees
- moved C5 44.3 mm to (72.8, 108.1), turned to 90 degrees
- moved U2 43.1 mm to (88.8, 108.1)
- moved U3 43.0 mm to (78.9, 108.1)
- moved R3 34.2 mm to (108.6, 119.3), turned to 0 degrees
- moved R4 34.2 mm to (98.7, 119.3), turned to 0 degrees
- moved C4 32.3 mm to (84.8, 108.1), turned to -90 degrees
- moved A1 28.9 mm to (139.6, 78.4)
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Connections:
- A1 pad 1: unconnected-(A1-D1/TX-Pad1) -> /RX/D1
- A1 pad 10: BTN2 -> /BTN2
- A1 pad 11: Sens0 -> /Sens0
- A1 pad 12: Sens1 -> /Sens1
- A1 pad 13: Servo -> /Servo
- A1 pad 14: MA1 -> /MA1
- A1 pad 15: Sens2 -> /Sens2
- A1 pad 16: Sens3 -> /Sens3
- A1 pad 19: Sens4 -> /Sens4
- A1 pad 2: unconnected-(A1-D0/RX-Pad2) -> /TX/D0
- A1 pad 20: Sens5 -> /Sens5
- A1 pad 21: Sens6 -> /Sens6
- A1 pad 22: Sens7 -> /Sens7
- A1 pad 23: SDA -> /SDA
- A1 pad 24: SCL -> /SCL
- A1 pad 25: Sens8 -> /Sens8
- A1 pad 26: Sens9 -> /Sens9
- A1 pad 27: +5V -> unconnected-(A1-+5V-Pad27)
- A1 pad 28: unconnected-(A1-~{RESET}-Pad28) -> Net-(A1-~{RESET}-Pad28)
- A1 pad 3: unconnected-(A1-~{RESET}-Pad3) -> Net-(A1-~{RESET}-Pad28)
- A1 pad 30: VCC -> +5V
- A1 pad 5: BTN1 -> /BTN1
- A1 pad 6: MB1 -> /MB1
- A1 pad 7: GO -> /Go
- A1 pad 8: MB2 -> /MB2
- A1 pad 9: MA2 -> /MA2
- C1 pad 1: VM -> +BATT
- C2 pad 1: VCC -> +5V
- C3 pad 1: VM -> +BATT
- C4 pad 1: VM -> GND
- C4 pad 2: GND -> +BATT
- C5 pad 1: VM -> +BATT
- C6 pad 1: VM -> +BATT
- R1 pad 2: BTN1 -> /BTN2
- R2 pad 2: BTN2 -> /BTN1
- R3 pad 1: GND -> Net-(U2-ILIM)
- R3 pad 2: Net-(U2-ILIM) -> GND
- R4 pad 1: GND -> Net-(U3-ILIM)
- R4 pad 2: Net-(U3-ILIM) -> GND
- SW2 pad 1: BTN1 -> /BTN2
- SW3 pad 1: BTN2 -> /BTN1
- SW4 pad 1: Net-(J1-Pin_2) -> Net-(A1-~{RESET}-Pad28)
- SW4 pad 2: VM -> GND
- U1 pad 1: VM -> +BATT
- U1 pad 3: VCC -> +5V
- U2 pad 2: MB1 -> /MA2
- U2 pad 3: MB2 -> /MA1
- U2 pad 5: VM -> +BATT
- U3 pad 2: MA1 -> /MB2
- U3 pad 3: MA2 -> /MB1
- U3 pad 5: VM -> +BATT
Routing:
- net +5V: track 182.0 -> 0.00 mm, vias 2 -> 0
- net GND: track 104.2 -> 0.00 mm, vias 10 -> 0
- net +3.3V: track 74.5 -> 0.00 mm, vias 1 -> 0
- net VCC: track 72.5 -> 0.00 mm, vias 2 -> 0
- net Sens0: track 70.2 -> 0.00 mm
- net Sens2: track 65.2 -> 0.00 mm
- net Sens1: track 65.2 -> 0.00 mm
- net MA1: track 64.4 -> 0.00 mm, vias 1 -> 0
- net VM: track 57.1 -> 0.00 mm, vias 2 -> 0
- net MA2: track 55.1 -> 0.00 mm, vias 1 -> 0
- net BTN2: track 51.6 -> 0.00 mm
- net MB2: track 42.7 -> 0.00 mm, vias 1 -> 0
- net MB1: track 38.5 -> 0.00 mm, vias 1 -> 0
- net BTN1: track 28.8 -> 0.00 mm
- net SDA: track 27.2 -> 0.00 mm, vias 1 -> 0
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- removed copper zone on B.Cu, net GND
- removed copper zone on F.Cu, net GND
Other:
- board size 85.5 x 24 mm -> 86 x 25 mm
- board text added: "TENN Rev3.0 by tenn.bots"
- board text removed: "3.3V"
- board text removed: "5V"
- board text removed: "A0"
- board text removed: "A1"
- board text removed: "A2"
- board text removed: "A3"
- board text removed: "A6"
- board text removed: "A7"
- board text removed: "D12"
- board text removed: "D13"
- board text removed: "D8"
- board text removed: "D9"
- board text removed: "GND"
- board text removed: "TENN Rev2.2 by tenn.bots"
