File: PCBS/Boards/Tei/Tei.kicad_pcb (KiCad board)
At the start: 2 copper layers, 85.5 x 32.5 mm, 37 parts, among them J1 Conn_01x02_Socket, J12 Conn_01x03_Pin, J13 Conn_01x02_Socket, J14 Conn_01x02_Socket, J2 Conn_01x03_Pin, J3 Conn_01x03_Pin, J4 Conn_01x03_Pin, J5 Conn_01x03_Pin, J6 Conn_01x03_Pin, J7 Conn_01x03_Pin, J8 Conn_01x03_Pin, J9 Conn_01x03_Pin, SW1 SW_SPDT, SW2 SW_Coded_SH-7010, U1 TB6612FNG, U2 AMS1117-5.0

Commit message: updates files for Tamashii
Routing:
- net +5V: track 203.0 -> 209.4 mm
