File: PCBS/Boards/Tei/Tei.kicad_sch (KiCad schematic)
At the start: 34 parts, among them J1 Conn_01x02_Socket, J10 Conn_01x04_Socket, J11 Conn_01x04_Socket, J12 Conn_01x03_Pin, J13 Conn_01x02_Socket, J14 Conn_01x02_Socket, J2 Conn_01x03_Pin, J3 Conn_01x03_Pin, J4 Conn_01x03_Pin, J5 Conn_01x03_Pin, J6 Conn_01x03_Pin, J7 Conn_01x03_Pin, J8 Conn_01x03_Pin, J9 Conn_01x03_Pin, SW1 SW_SPDT, SW3 SW_Coded_SH-7010, U1 TB6612FNG, U2 AMS1117-5.0

Commit message: updated readme and PCB files
Changed lines of the file:
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@@
 (kicad_sch
-	(version 20231120)
+	(version 20250114)
 	(generator "eeschema")
-	(generator_version "8.0")
+	(generator_version "9.0")
 	(paper "A4")
 	(title_block
@@
 		(comment 2 "@tenn.bots")
 	)
+	(text "Remote Connector"
+		(exclude_from_sim no)
+		(at 63.5 97.155 0)
+		(effects
+			(font
+				(size 1.27 1.27)
+				(bold yes)
+			)
+			(justify left bottom)
+		)
+	)
+	(text "Arduino and Rotary Coded Switch"
+		(exclude_from_sim no)
+		(at 101.6 71.755 0)
+		(effects
+			(font
+				(size 1.27 1.27)
+				(thickness 0.254)
+				(bold yes)
+			)
+			(justify left bottom)
+		)
+	)
+	(text "Sensor Connectors"
+		(exclude_from_sim no)
+		(at 38.1 71.755 0)
+		(effects
+			(font
+				(size 1.27 1.27)
+				(thickness 0.254)
+				(bold yes)
+			)
+			(justify left bottom)
+		)
+	)
+	(text "Test Headers"
+		(exclude_from_sim no)
+		(at 63.5 122.555 0)
+		(effects
+			(font
+				(size 1.27 1.27)
+				(bold yes)
+			)
+			(justify left bottom)
+		)
+	)
+	(text "Bluetooth Module Connector"
+		(exclude_from_sim no)
+		(at 63.5 71.755 0)
+		(effects
+			(font
+				(size 1.27 1.27)
+				(bold yes)
+			)
+			(justify left bottom)
+		)
+	)
+	(text "Power Supply and Voltage Regulator"
+		(exclude_from_sim no)
+		(at 38.1 40.005 0)
+		(effects
+			(font
+				(size 1.27 1.27)
+				(thickness 0.254)
+				(bold yes)
+			)
+			(justify left bottom)
+		)
+	)
+	(text "Power LED"
+		(exclude_from_sim no)
+		(at 101.6 40.005 0)
+		(effects
+			(font
+				(size 1.27 1.27)
+				(bold yes)
+			)
+			(justify left bottom)
+		)
+	)
+	(text "Motor Driver"
+		(exclude_from_sim no)
+		(at 196.85 71.755 0)
+		(effects
+			(font
+				(size 1.27 1.27)
+				(thickness 0.254)
+				(bold yes)
+			)
+			(justify left bottom)
+		)
+	)
 	(junction
 		(at 132.715 130.81)
@@
 		)
 	)
-	(text "Remote Connector"
-		(exclude_from_sim no)
-		(at 63.5 97.155 0)
-		(effects
-			(font
-				(size 1.27 1.27)
-				(bold yes)
-			)
-			(justify left bottom)
-		)
-	)
-	(text "Arduino and Rotary Coded Switch"
-		(exclude_from_sim no)
-		(at 101.6 71.755 0)
-		(effects
-			(font
-				(size 1.27 1.27)
-				(thickness 0.254)
-				(bold yes)
-			)
-			(justify left bottom)
-		)
-	)
-	(text "Sensor Connectors"
-		(exclude_from_sim no)
-		(at 38.1 71.755 0)
-		(effects
-			(font
-				(size 1.27 1.27)
-				(thickness 0.254)
-				(bold yes)
-			)
-			(justify left bottom)
-		)
-	)
-	(text "Test Headers"
-		(exclude_from_sim no)
-		(at 63.5 122.555 0)
-		(effects
-			(font
-				(size 1.27 1.27)
-				(bold yes)
-			)
-			(justify left bottom)
-		)
-	)
-	(text "Bluetooth Module Connector"
-		(exclude_from_sim no)
-		(at 63.5 71.755 0)
-		(effects
-			(font
-				(size 1.27 1.27)
-				(bold yes)
-			)
-			(justify left bottom)
-		)
-	)
-	(text "Power Supply and Voltage Regulator"
-		(exclude_from_sim no)
-		(at 38.1 40.005 0)
-		(effects
-			(font
-				(size 1.27 1.27)
-				(thickness 0.254)
-				(bold yes)
-			)
-			(justify left bottom)
-		)
-	)
-	(text "Power LED"
-		(exclude_from_sim no)
-		(at 101.6 40.005 0)
-		(effects
-			(font
-				(size 1.27 1.27)
-				(bold yes)
-			)
-			(justify left bottom)
-		)
-	)
-	(text "Motor Driver"
-		(exclude_from_sim no)
-		(at 196.85 71.755 0)
-		(effects
-			(font
-				(size 1.27 1.27)
-				(thickness 0.254)
-				(bold yes)
-			)
-			(justify left bottom)
-		)
-	)
 	(global_label "MA2"
 		(shape input)
@@
 		)
 	)
+	(embedded_fonts no)
 )
