File: PCBS/Boards/Ma/Ma/Ma.kicad_pcb (KiCad board)
At the start: 2 copper layers, 50 x 30 mm, 43 parts, among them J1 Conn_01x02_Socket, J10 Conn_01x14_Pin, J2 Conn_01x04_Socket, J3 Conn_01x02_Pin, J4 Conn_01x02_Pin, J5 Conn_01x03_Pin, J7 Conn_01x03_Pin, J8 Conn_01x06_Socket, J9 Conn_01x04_Socket, SW1 SW_Push, SW2 SW_SPDT, SW3 SW_Push, SW4 SW_Push, U1 ATmega328P-M, Y1 Crystal

Commit message: created SHU BEC, added KiCad project files and production files
Parts:
- removed C1, C10, C13, C2, C3, C5: 0.1uF, Capacitor_SMD:C_0805_2012Metric
- removed C11, C12: 470uF, Capacitor_SMD:CP_Elec_8x10.5
- removed C4: 4.7uF, Capacitor_SMD:C_0805_2012Metric
- removed D1, D2: LED, LED_SMD:LED_0603_1608Metric
- removed G*** (x4): LOGO, LOGO
- removed H1, H2, H3, H4: MountingHole, MountingHole:MountingHole_2.2mm_M2
- removed J1: Conn_01x02_Socket, Connector_AMASS:AMASS_XT30U-M_1x02_P5.0mm_Vertical
- removed J10: Conn_01x14_Pin, Connector_PinHeader_2.54mm:PinHeader_1x14_P2.54mm_Vertical
- removed J2, J9: Conn_01x04_Socket, Connector_PinSocket_2.54mm:PinSocket_1x04_P2.54mm_Vertical
- removed J3, J4: Conn_01x02_Pin, Connector_JST:JST_XH_B2B-XH-A_1x02_P2.50mm_Vertical
- removed J5: Conn_01x03_Pin, Package_TO_SOT_SMD:TO-252-2
- removed J7: Conn_01x03_Pin, EasyEDA:HDR-SMD_3P-P2.54-H-M-W13.3-N
- removed J8: Conn_01x06_Socket, EasyEDA:HDR-SMD_6P-P2.54-H-F-W11.7
- removed R1, R2, R3, R4, R5, R6, R7: R, Resistor_SMD:R_0603_1608Metric
- removed SW1: SW_Push, Button_Switch_SMD:SW_Push_SPST_NO_Alps_SKRK
- removed SW2: SW_SPDT, EasyEDA:SW-TH_XKB_SS-12M11XX
- removed SW3, SW4: SW_Push, Button_Switch_SMD:SW_SPST_PTS810
- removed U1: ATmega328P-M, Package_DFN_QFN:QFN-32-1EP_5x5mm_P0.5mm_EP3.1x3.1mm
- removed U3, U4: ~, Package_SO:SOP-8_3.9x4.9mm_P1.27mm
- removed Y1: Crystal, Crystal:Crystal_SMD_3215-2Pin_3.2x1.5mm
Routing:
- net +5V: track 141.9 -> 0.00 mm, vias 4 -> 0
- net +BATT: track 52.8 -> 0.00 mm
- net Reset: track 45.8 -> 0.00 mm, vias 1 -> 0
- net /BTN2: track 27.9 -> 0.00 mm
- net /BTN1: track 26.2 -> 0.00 mm
- net /START: track 25.7 -> 0.00 mm, vias 1 -> 0
- net /D13: track 24.0 -> 0.00 mm, vias 1 -> 0
- net /MB1: track 17.2 -> 0.00 mm, vias 2 -> 0
- net /A3: track 16.4 -> 0.00 mm
- net GND: track 16.4 -> 0.00 mm, vias 18 -> 0
- net /MB2: track 15.7 -> 0.00 mm, vias 2 -> 0
- net /SERVO: track 15.3 -> 0.00 mm, vias 1 -> 0
- net /SCL: track 14.8 -> 0.00 mm, vias 1 -> 0
- net /MA1: track 14.6 -> 0.00 mm, vias 2 -> 0
- net /SDA: track 14.3 -> 0.00 mm, vias 1 -> 0
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- removed copper zone on B.Cu, net GND
- removed copper zone on F.Cu, net GND
Other:
- board outline removed
- board text removed: "CROSSFIRE HURRICANE"
- board text removed: "If you can read this: STAY CURIOUS"
- board text removed: "MA V1 rev. 1.0 by tenn.bots"
