File: PCBS/Boards/Ma/Ma/Ma.kicad_sch (KiCad schematic)
At the start: 46 parts, among them J1 Conn_01x02_Socket, J2 Conn_01x06_Socket, J3 Conn_01x04_Socket, J4 Conn_01x14_Pin, J5 Conn_01x03_Pin, J6 Conn_01x04_Socket, J7 Conn_01x02_Pin, J8 Conn_01x02_Pin, Q1 PMOS, SW1 SW_SPDT, SW2 SW_Push, SW3 SW_Push, SW4 SW_Push, U1 XL1509-5.0, U2 ATmega328P-M, U3 RZ7899-MS, U4 RZ7899-MS, Y1 Crystal

Commit message: created SHU BEC, added KiCad project files and production files
Parts:
- removed U3, U4: RZ7899-MS, EasyEDA:SOIC-8_L4.9-W3.9-P1.27-LS6.0-BL, symbol EasyEDA:RZ7899-MS
- added U3, U4: rz7899, EasyEDA:SOP-8_L4.9-W3.9-P1.27-LS6.0-BL, symbol EasyEDA:rz7899
- D2: renamed from D1; footprint (none) -> Diode_SMD:D_SMC
- J2: footprint EasyEDA:HDR-SMD_6P-P2.54-H-F-W11.7 -> (none)
- J5: footprint EasyEDA:HDR-SMD_3P-P2.54-H-M-W13.3-N -> (none)
- SW1: footprint EasyEDA:SW-TH_XKB_SS-12M11XX -> (none)
- renumbered C4 to C1, C11 to C10, C10 to C11, C5 to C2, C6 to C3, C1 to C4, C7 to C5, C8 to C6, C2 to C7, C3 to C8, D3 to D1, D2 to D3, R3 to R2, R4 to R3, R5 to R4, R6 to R5, R2 to R6, U2 to U1, U1 to U2
Connections:
- net +5V: now also C2.2; no longer C2.1
- net +BATT: now also U3.4 (VCC), U4.4 (VCC)
- net -BATT: now also C2.1, U3.3 (GND), U4.3 (GND); no longer C2.2
- net MA1: now also U4.1 (BI)
- net MA2: now also U4.2 (FI)
- net MB1: now also U3.1 (BI)
- net MB2: now also U3.2 (FI)
- net at J7.1 (Pin_1): now also U3.5 (FO), U3.6 (FO)
- net at J7.2 (Pin_2): now also U3.7 (BO), U3.8 (BO)
- net at J8.1 (Pin_1): now also U4.5 (FO), U4.6 (FO)
- net at J8.2 (Pin_2): now also U4.7 (BO), U4.8 (BO)
Other:
- moved on the sheet: C1, C2, J2, J3, J4, J5, J6, R3
